Commit message: add for resilisilient planner

File: rotors_description/urdf/component_snippets.xacro (robot description, xacro)
@@ -682,5 +682,5 @@
       </visual>
       <inertial>
-        <mass value="0.13" />
+        <mass value="1e-5" />
         <origin xyz="0 0 0" rpy="0 0 0" />
         <inertia ixx="1e-6" ixy="0" ixz="0" iyy="1e-6" iyz="0" izz="1e-6" />

File: rotors_description/urdf/hummingbird.xacro (robot description, xacro)
@@ -54,4 +54,5 @@
     body_height="${body_height}"
     use_mesh_file="${use_mesh_file}"
+    color="Grey"
     mesh_file="${mesh_file}">
     <xacro:insert_block name="body_inertia" />

File: rotors_description/urdf/multirotor_base.xacro (robot description, xacro)
@@ -31,7 +31,7 @@
     </inertial>
   </xacro:macro>
-  <!-- Main multirotor link -->
+<!-- Main multirotor link -->
   <xacro:macro name="multirotor_base_macro"
-    params="robot_namespace mass body_width body_height use_mesh_file mesh_file *inertia">
+    params="robot_namespace mass body_width body_height use_mesh_file color mesh_file *inertia">
     <link name="${robot_namespace}/base_link"></link>
     <joint name="${robot_namespace}/base_joint" type="fixed">
